File: Board/Power Module Rev 5/CanBus.kicad_sch (KiCad schematic)
At the start: 4 parts, among them U11 MCP2558FD-xMF

Commit message: Board Progress
Connections:
- net CanHi renamed Can+
- net CanLo renamed Can-
Changed lines of the file:
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@@
     )
   )
-  (global_label "CanLo" (shape input) (at 184.15 80.01 0) (fields_autoplaced)
+  (global_label "Can-" (shape input) (at 184.15 80.01 0) (fields_autoplaced)
     (effects (font (size 1.27 1.27)) (justify left))
-    (property "Intersheetrefs" "${INTERSHEET_REFS}" (at 192.8009 80.01 0)
+    (property "Intersheetrefs" "${INTERSHEET_REFS}" (at 192.1962 80.01 0)
       (effects (font (size 1.27 1.27)) (justify left) hide)
     )
   )
-  (global_label "CanHi" (shape input) (at 184.15 74.93 0) (fields_autoplaced)
+  (global_label "Can+" (shape input) (at 184.15 74.93 0) (fields_autoplaced)
     (effects (font (size 1.27 1.27)) (justify left))
-    (property "Intersheetrefs" "${INTERSHEET_REFS}" (at 192.5591 74.93 0)
+    (property "Intersheetrefs" "${INTERSHEET_REFS}" (at 192.1962 74.93 0)
       (effects (font (size 1.27 1.27)) (justify left) hide)
     )

Commit message: Board Update
Connections:
- net Can+: now also D1.1 (C1); no longer D1.2 (C2)
- net Can-: now also D1.2 (C2); no longer D1.1 (C1)
Changed lines of the file:
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@@
 (kicad_sch (version 20230121) (generator eeschema)
   (paper "A4")
-  (junction (at 165.1 74.93) (diameter 0) (color 0 0 0 0)
-  )
-  (junction (at 170.18 80.01) (diameter 0) (color 0 0 0 0)
+  (junction (at 165.1 80.01) (diameter 0) (color 0 0 0 0)
   )
   (junction (at 111.76 80.01) (diameter 0) (color 0 0 0 0)
@@
   (junction (at 143.51 50.8) (diameter 0) (color 0 0 0 0)
   )
+  (junction (at 170.18 74.93) (diameter 0) (color 0 0 0 0)
+  )
   (wire (pts (xy 128.27 72.39) (xy 130.81 72.39))
     (stroke (width 0) (type default))
   )
   (wire (pts (xy 154.94 50.8) (xy 143.51 50.8))
+    (stroke (width 0) (type default))
+  )
+  (wire (pts (xy 165.1 80.01) (xy 184.15 80.01))
     (stroke (width 0) (type default))
   )
@@
     (stroke (width 0) (type default))
   )
-  (wire (pts (xy 165.1 74.93) (xy 184.15 74.93))
+  (wire (pts (xy 170.18 74.93) (xy 184.15 74.93))
+    (stroke (width 0) (type default))
+  )
+  (wire (pts (xy 156.21 74.93) (xy 170.18 74.93))
+    (stroke (width 0) (type default))
+  )
+  (wire (pts (xy 165.1 80.01) (xy 165.1 83.82))
     (stroke (width 0) (type default))
   )
@@
     (stroke (width 0) (type default))
   )
-  (wire (pts (xy 170.18 80.01) (xy 170.18 83.82))
-    (stroke (width 0) (type default))
-  )
   (wire (pts (xy 128.27 74.93) (xy 130.81 74.93))
     (stroke (width 0) (type default))
@@
     (stroke (width 0) (type default))
   )
-  (wire (pts (xy 156.21 74.93) (xy 165.1 74.93))
-    (stroke (width 0) (type default))
-  )
-  (wire (pts (xy 156.21 80.01) (xy 170.18 80.01))
-    (stroke (width 0) (type default))
-  )
   (wire (pts (xy 111.76 91.44) (xy 111.76 93.98))
     (stroke (width 0) (type default))
   )
-  (wire (pts (xy 165.1 74.93) (xy 165.1 83.82))
+  (wire (pts (xy 111.76 80.01) (xy 111.76 86.36))
     (stroke (width 0) (type default))
   )
-  (wire (pts (xy 111.76 80.01) (xy 111.76 86.36))
+  (wire (pts (xy 170.18 74.93) (xy 170.18 83.82))
     (stroke (width 0) (type default))
   )
@@
     (stroke (width 0) (type default))
   )
-  (wire (pts (xy 170.18 80.01) (xy 184.15 80.01))
+  (wire (pts (xy 156.21 80.01) (xy 165.1 80.01))
     (stroke (width 0) (type default))
   )
