File: Board/Power Module Rev 5/Mcu.kicad_sch (KiCad schematic)
At the start: 4 parts, among them J4 Conn_ARM_SWD_TagConnect_TC203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, J4 USB_C_Receptacle_USB2.0, U1 STM32G491CCUx, U6 MB85RS64

Commit message: Board Update
Parts:
- removed U1: STM32G491CCUx, Package_DFN_QFN:QFN-48-1EP_7x7mm_P0.5mm_EP5.6x5.6mm, symbol MCU_ST_STM32G4:STM32G491CCUx
- added C13 (x4): ~, Capacitor_SMD:C_0603_1608Metric_Pad1.08x0.95mm_HandSolder, symbol Device:C_Small
- added FB1: FerriteBead_Small, Resistor_SMD:R_0603_1608Metric_Pad0.98x0.95mm_HandSolder, symbol Device:FerriteBead_Small
- added R1 (x2): 5.1K, Resistor_SMD:R_0603_1608Metric_Pad0.98x0.95mm_HandSolder, symbol Device:R_Small
- added U17: STM32G491CEUx, Package_DFN_QFN:QFN-48-1EP_7x7mm_P0.5mm_EP5.6x5.6mm, symbol MCU_ST_STM32G4:STM32G491CEUx
- added Y1, Y2: Crystal_Small, Crystal:Crystal_SMD_5032-2Pin_5.0x3.2mm, symbol Device:Crystal_Small
- J4: footprint (none) -> Connector_USB:USB_C_Receptacle_JAE_DX07S016JA1R1500
Connections:
- net CanRx: now also U17.43 (PB5)
- net CanSilent: now also U17.39 (PC10)
- net CanTx: now also U17.44 (PB6)
- net Den7-8: now also U17.28 (PB15)
- net Dsel7-8: now also U17.26 (PB13)
- net Is1: now also U17.8 (PA0)
- net Is2: now also U17.9 (PA1)
- net Is3: now also U17.10 (PA2)
- net Is4: now also U17.11 (PA3)
- net Is5: now also U17.18 (PB1)
- net Is6: now also U17.24 (PB11)
- net Is7-8: now also U17.25 (PB12)
- net Is9-10: now also U17.27 (PB14)
- net L6699-Int: now also U17.42 (PB4)
- net L6699-Rst: now also U17.40 (PC11)
- net L6699-Sync: now also U17.2 (PC13)
- net Power Switch Status: now also U17.38 (PA15)
- net Pwm_Ctr_Enable: now also U17.32 (PA10)
- net SCL: now also U17.31 (PA9)
- net SDA: now also U17.30 (PA8)
- net Usb 5V: now also J4.A4 (VBUS), J4.A9 (VBUS), J4.B4 (VBUS), J4.B9 (VBUS)
- net GND: now reaches J4.A1 (GND), J4.A12 (GND), J4.B1 (GND), J4.B12 (GND)
- net GND: now also J4.5 (GND), C13.1, C13.1, C13.1, C13.1, R1.2, R1.2, U17.49 (VSS)
- net at J4.A5 (CC1): now also R1.1
- net Usb D+: now reaches J4.A6 (D+)
- net Usb D+: now also J4.B6 (D+), U17.34 (PA12)
- net Usb D-: now reaches J4.A7 (D-)
- net Usb D-: now also J4.B7 (D-), U17.33 (PA11)
- net at J4.B5 (CC2): now also R1.1
- net +3.3V: now reaches J4.1 (VCC)
- net +3.3V: now also FB1.1, U17.1 (VBAT), U17.23 (VDD), U17.35 (VDD), U17.48 (VDD)
- net SWDIO: now reaches J4.2 (SWDIO)
- net SWDIO: now also U17.36 (PA13)
- net RESET: now reaches J4.3 (~{RESET})
- net RESET: now also U17.7 (PG10)
- net SWCLK: now reaches J4.4 (SWCLK)
- net SWCLK: now also U17.37 (PA14)
- net SWO: now reaches J4.6 (SWO)
- net SWO: now also U17.41 (PB3)
- new net: C13.2, U17.4 (PC15), Y2.1
- new net: C13.2, U17.3 (PC14), Y2.2
- new net: C13.2, U17.6 (PF1), Y1.1
- new net: FB1.2, U17.21 (VDDA)
- new net: C13.2, U17.5 (PF0), Y1.2
- new net BOOT_0: U17.46 (PB8)
- new net Den2: U17.47 (PB9)
- new net Den5: U17.22 (PB10)
- new net SPI1_Miso: U17.14 (PA6)
- new net SPI1_Mosi: U17.15 (PA7)
- new net SPI1_SS1: U17.12 (PA4)
- new net SPI1_SS2: U17.17 (PB0)
- new net SPI1_Sclk: U17.13 (PA5)
- no-connect marks 0 -> 3
Other:
- moved on the sheet: J4

Commit message: Board Update
Parts:
- added C13 (x4), C34: 0.1uF, Capacitor_SMD:C_0603_1608Metric_Pad1.08x0.95mm_HandSolder, symbol Device:C_Small
- added C13: 1uF, Capacitor_SMD:C_0603_1608Metric_Pad1.08x0.95mm_HandSolder, symbol Device:C_Small
- added C13: 10nF, Capacitor_SMD:C_0603_1608Metric_Pad1.08x0.95mm_HandSolder, symbol Device:C_Small
- added R1: 10K, Resistor_SMD:R_0603_1608Metric_Pad0.98x0.95mm_HandSolder, symbol Device:R_Small
- added S1, S2: B3U-1000P, digikey-footprints:Switch_Tactile_SMD_B3U-1000P, symbol dk_Tactile-Switches:B3U-1000P
- U17: footprint Package_DFN_QFN:QFN-48-1EP_7x7mm_P0.5mm_EP5.6x5.6mm -> Package_DFN_QFN:QFN-48-1EP_7x7mm_P0.5mm_EP5.6x5.6mm_ThermalVias
- U6: footprint (none) -> Package_SO:SSOP-8_3.9x5.05mm_P1.27mm
Connections:
- net +3.3V: now also U6.8 (VDD), C13.2, C13.2, C13.2, C13.2, C13.2, C13.2, C34.1, S2.2
- net BOOT_0: now also R1.1, S2.1
- net CanSilent: now also U17.2 (PC13); no longer U17.39 (PC10)
- net Den2: now also U17.28 (PB15); no longer U17.47 (PB9)
- net Den5: now also U17.38 (PA15); no longer U17.22 (PB10)
- net Den7-8: now also U17.32 (PA10); no longer U17.28 (PB15)
- net Dsel7-8: now also U17.29 (PC6); no longer U17.26 (PB13)
- net GND: now also U6.4 (GND), C13.1, C13.1, C13.1, C13.1, C13.1, C13.1, C34.2, R1.2, S1.2
- net Is1: now also U17.27 (PB14); no longer U17.8 (PA0)
- net Is2: now also U17.24 (PB11); no longer U17.9 (PA1)
- net Is4: now also U17.9 (PA1); no longer U17.11 (PA3)
- net Is5: now also U17.25 (PB12); no longer U17.18 (PB1)
- net Is6: now also U17.11 (PA3); no longer U17.24 (PB11)
- net Is7-8: now also U17.18 (PB1); no longer U17.25 (PB12)
- net Is9-10: now also U17.8 (PA0); no longer U17.27 (PB14)
- net L6699-Sync: now also U17.45 (PB7); no longer U17.2 (PC13)
- net Power Switch Status: now also U17.19 (PB2); no longer U17.38 (PA15)
- net Pwm_Ctr_Enable: now also U17.47 (PB9); no longer U17.32 (PA10)
- net RESET: now also S1.1
- net SPI1_Miso: now also U6.2 (SO)
- net SPI1_Mosi: now also U6.5 (SI)
- net SPI1_SS1: now also U17.39 (PC10); no longer U17.12 (PA4)
- net SPI1_SS2: now also U17.16 (PC4), U6.1 (~{CS}); no longer U17.17 (PB0)
- net SPI1_Sclk: now also U6.6 (SCK)
- net Memory_Wp: now reaches U6.3 (~{WP})
- net Memory_Wp: now also U17.17 (PB0)
- net Memory_Hold: now reaches U6.7 (~{HOLD})
- net Memory_Hold: now also U17.12 (PA4)
Other:
- note added: "Vdda"
- moved on the sheet: J4

Commit message: Update Board
Parts:
- added FB2: FerriteBead_Small, Resistor_SMD:R_0603_1608Metric_Pad0.98x0.95mm_HandSolder, symbol Device:FerriteBead_Small
Connections:
- net GND: now also FB2.2
- net Usb_Shield: now reaches J4.S1 (SHIELD)
- net Usb_Shield: now also FB2.1
- no-connect marks 3 -> 2
Changed lines of the file:
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@@
 (kicad_sch (version 20230121) (generator eeschema)
   (paper "A4")
+  (junction (at 220.98 77.47) (diameter 0) (color 0 0 0 0)
+  )
   (junction (at 71.12 74.93) (diameter 0) (color 0 0 0 0)
   )
@@
   )
   (no_connect (at 236.22 62.23))
-  (no_connect (at 213.36 69.85))
   (no_connect (at 236.22 59.69))
   (wire (pts (xy 147.32 26.67) (xy 147.32 30.48))
@@
     (stroke (width 0) (type default))
   )
+  (wire (pts (xy 220.98 69.85) (xy 220.98 77.47))
+    (stroke (width 0) (type default))
+  )
   (wire (pts (xy 58.42 49.53) (xy 60.96 49.53))
     (stroke (width 0) (type default))
@@
     (stroke (width 0) (type default))
   )
+  (wire (pts (xy 213.36 69.85) (xy 213.36 71.12))
+    (stroke (width 0) (type default))
+  )
   (wire (pts (xy 236.22 36.83) (xy 269.24 36.83))
     (stroke (width 0) (type default))
@@
     (stroke (width 0) (type default))
   )
+  (wire (pts (xy 213.36 77.47) (xy 220.98 77.47))
+    (stroke (width 0) (type default))
+  )
   (wire (pts (xy 157.48 30.48) (xy 147.32 30.48))
     (stroke (width 0) (type default))
@@
     (stroke (width 0) (type default))
   )
+  (wire (pts (xy 213.36 76.2) (xy 213.36 77.47))
+    (stroke (width 0) (type default))
+  )
   (wire (pts (xy 166.37 40.64) (xy 157.48 40.64))
     (stroke (width 0) (type default))
@@
   )
   (wire (pts (xy 147.32 38.1) (xy 147.32 40.64))
+    (stroke (width 0) (type default))
+  )
+  (wire (pts (xy 220.98 77.47) (xy 220.98 80.01))
     (stroke (width 0) (type default))
   )
@@
   )
   (label "SPI1_SS2" (at 85.09 58.42 180) (fields_autoplaced)
+    (effects (font (size 1.27 1.27)) (justify right bottom))
+  )
+  (label "Usb_Shield" (at 213.36 71.12 180) (fields_autoplaced)
     (effects (font (size 1.27 1.27)) (justify right bottom))
   )
@@
     )
   )
-  (symbol (lib_id "power:GND") (at 220.98 69.85 0) (unit 1)
-    (in_bom yes) (on_board yes) (dnp no)
-    (property "Reference" "#PWR018" (at 220.98 76.2 0)
-      (effects (font (size 1.27 1.27)) hide)
-    )
-    (property "Value" "GND" (at 221.107 74.2442 0)
+  (symbol (lib_id "Device:FerriteBead_Small") (at 213.36 73.66 0) (unit 1)
+    (in_bom yes) (on_board yes) (dnp no) (fields_autoplaced)
+    (property "Reference" "FB2" (at 215.9 72.9869 0)
+      (effects (font (size 1.27 1.27)) (justify left))
+    )
+    (property "Value" "FerriteBead_Small" (at 215.9 75.5269 0)
+      (effects (font (size 1.27 1.27)) (justify left))
+    )
+    (property "Footprint" "Resistor_SMD:R_0603_1608Metric_Pad0.98x0.95mm_HandSolder" (at 211.582 73.66 90)
+      (effects (font (size 1.27 1.27)) hide)
+    )
+    (property "Datasheet" "~" (at 213.36 73.66 0)
+      (effects (font (size 1.27 1.27)) hide)
+    )
+    (pin "1")
+    (pin "2")
+    (instances
+      (project "Power Module Rev 5"
+        (path "/678ed6a7-73b5-414a-90da-5837647f5dd4/a3a78077-6b53-4c9d-ba53-5da8cf684a1d"
+          (reference "FB2") (unit 1)
+        )
+      )
+    )
+  )
+  (symbol (lib_id "power:GND") (at 220.98 80.01 0) (unit 1)
+    (in_bom yes) (on_board yes) (dnp no)
+    (property "Reference" "#PWR018" (at 220.98 86.36 0)
+      (effects (font (size 1.27 1.27)) hide)
+    )
+    (property "Value" "GND" (at 221.107 84.4042 0)
       (effects (font (size 1.27 1.27)))
     )
-    (property "Footprint" "" (at 220.98 69.85 0)
-      (effects (font (size 1.27 1.27)) hide)
-    )
-    (property "Datasheet" "" (at 220.98 69.85 0)
-      (effects (font (size 1.27 1.27)) hide)
-    )
+    (property "Footprint" "" (at 220.98 80.01 0)
+      (effects (font (size 1.27 1.27)) hide)
+    )
+    (property "Datasheet" "" (at 220.98 80.01 0)
+      (effects (font (size 1.27 1.27)) hide)
+    )

Commit message: Update config and renames on schematic
Connections:
- net Power Switch Status renamed PowerSwitchStatus
- net SPI1_SS1 renamed SPI1_SS_L9966
- net SPI1_SS2 renamed SPI1_SS_Memory
Changed lines of the file:
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@@
     (effects (font (size 1.27 1.27)) (justify right bottom))
   )
-  (label "SPI1_SS2" (at 85.09 58.42 180) (fields_autoplaced)
+  (label "SPI1_SS_Memory" (at 85.09 58.42 180) (fields_autoplaced)
     (effects (font (size 1.27 1.27)) (justify right bottom))
   )
@@
     (effects (font (size 1.27 1.27)) (justify left bottom))
   )
-  (label "SPI1_SS2" (at 189.23 130.81 180) (fields_autoplaced)
+  (label "SPI1_SS_Memory" (at 189.23 130.81 180) (fields_autoplaced)
     (effects (font (size 1.27 1.27)) (justify right bottom))
   )
@@
     )
   )
-  (global_label "Power Switch Status" (shape input) (at 85.09 83.82 180) (fields_autoplaced)
+  (global_label "PowerSwitchStatus" (shape input) (at 85.09 83.82 180) (fields_autoplaced)
     (effects (font (size 1.27 1.27)) (justify right))
-    (property "Intersheetrefs" "${INTERSHEET_REFS}" (at 62.9408 83.82 0)
+    (property "Intersheetrefs" "${INTERSHEET_REFS}" (at 64.4648 83.82 0)
       (effects (font (size 1.27 1.27)) (justify right) hide)
     )
@@
     )
   )
-  (global_label "SPI1_SS1" (shape input) (at 85.09 63.5 180) (fields_autoplaced)
+  (global_label "SPI1_SS_L9966" (shape input) (at 85.09 63.5 180) (fields_autoplaced)
     (effects (font (size 1.27 1.27)) (justify right))
-    (property "Intersheetrefs" "${INTERSHEET_REFS}" (at 73.2943 63.5 0)
+    (property "Intersheetrefs" "${INTERSHEET_REFS}" (at 67.6701 63.5 0)
       (effects (font (size 1.27 1.27)) (justify right) hide)
     )

Commit message: Board Update
Parts:
- added D2: LED_Small, LED_SMD:LED_0603_1608Metric_Pad1.05x0.95mm_HandSolder, symbol Device:LED_Small
- added R1: 65, Resistor_SMD:R_0603_1608Metric_Pad0.98x0.95mm_HandSolder, symbol Device:R_Small
Connections:
- net GND: now also D2.1 (K)
- net User_Led: now reaches U17.22 (PB10)
- net User_Led: now also R1.1
- new net: D2.2 (A), R1.2
Changed lines of the file:
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@@
+    (stroke (width 0) (type default))
+  )
+  (wire (pts (xy 55.88 104.14) (xy 85.09 104.14))
     (stroke (width 0) (type default))
   )
@@
     (stroke (width 0) (type default))
   )
+  (wire (pts (xy 43.18 104.14) (xy 40.64 104.14))
+    (stroke (width 0) (type default))
+  )
   (wire (pts (xy 97.79 22.86) (xy 97.79 29.21))
     (stroke (width 0) (type default))
   )
+  (wire (pts (xy 48.26 104.14) (xy 50.8 104.14))
+    (stroke (width 0) (type default))
+  )
   (wire (pts (xy 102.87 29.21) (xy 100.33 29.21))
     (stroke (width 0) (type default))
@@
   )
   (wire (pts (xy 111.76 179.07) (xy 111.76 181.61))
+    (stroke (width 0) (type default))
+  )
+  (wire (pts (xy 40.64 104.14) (xy 40.64 106.68))
     (stroke (width 0) (type default))
   )
@@
   (label "Memory_Wp" (at 85.09 78.74 180) (fields_autoplaced)
     (effects (font (size 1.27 1.27)) (justify right bottom))
+  )
+  (label "User_Led" (at 57.15 104.14 0) (fields_autoplaced)
+    (effects (font (size 1.27 1.27)) (justify left bottom))
   )
   (label "SWCLK" (at 66.04 173.99 0) (fields_autoplaced)
@@
         (path "/678ed6a7-73b5-414a-90da-5837647f5dd4/a3a78077-6b53-4c9d-ba53-5da8cf684a1d"
           (reference "#PWR082") (unit 1)
+        )
+      )
+    )
+  )
+  (symbol (lib_id "power:GND") (at 40.64 106.68 0) (unit 1)
+    (in_bom yes) (on_board yes) (dnp no)
+    (property "Reference" "#PWR018" (at 40.64 113.03 0)
+      (effects (font (size 1.27 1.27)) hide)
+    )
+    (property "Value" "GND" (at 40.767 111.0742 0)
+      (effects (font (size 1.27 1.27)))
+    )
+    (property "Footprint" "" (at 40.64 106.68 0)
+      (effects (font (size 1.27 1.27)) hide)
+    )
+    (property "Datasheet" "" (at 40.64 106.68 0)
+      (effects (font (size 1.27 1.27)) hide)
+    )
+    (pin "1")
+    (instances
+      (project "Power Module Rev 4"
+        (path "/2f7b63dd-ee4f-415a-a7fc-f5e5e0f90b8a"
+          (reference "#PWR018") (unit 1)
+        )
+      )
+      (project "Power Module Rev 5"
+        (path "/678ed6a7-73b5-414a-90da-5837647f5dd4/ba6f5248-4cb0-41f9-9534-0fba5bdbe75a"
+          (reference "#PWR016") (unit 1)
+        )
+        (path "/678ed6a7-73b5-414a-90da-5837647f5dd4/a3a78077-6b53-4c9d-ba53-5da8cf684a1d"
+          (reference "#PWR093") (unit 1)
         )
       )
@@
     )
   )
+  (symbol (lib_id "Device:R_Small") (at 53.34 104.14 270) (unit 1)
+    (in_bom yes) (on_board yes) (dnp no) (fields_autoplaced)
+    (property "Reference" "R1" (at 53.34 99.06 90)
+      (effects (font (size 1.27 1.27)))
+    )
+    (property "Value" "65" (at 53.34 101.6 90)
+      (effects (font (size 1.27 1.27)))
+    )
+    (property "Footprint" "Resistor_SMD:R_0603_1608Metric_Pad0.98x0.95mm_HandSolder" (at 53.34 104.14 0)
+      (effects (font (size 1.27 1.27)) hide)
+    )
+    (property "Datasheet" "~" (at 53.34 104.14 0)
+      (effects (font (size 1.27 1.27)) hide)
+    )
+    (pin "1")
+    (pin "2")
+    (instances
+      (project "Power Module Rev 5"
+        (path "/678ed6a7-73b5-414a-90da-5837647f5dd4/ba6f5248-4cb0-41f9-9534-0fba5bdbe75a/28927523-0fd3-4824-a72b-28dbb4627c61"
+          (reference "R1") (unit 1)
+        )
+        (path "/678ed6a7-73b5-414a-90da-5837647f5dd4/ba6f5248-4cb0-41f9-9534-0fba5bdbe75a/2112056d-5440-4876-9be3-a7dbbd0302bd"
+          (reference "R2") (unit 1)
+        )
+        (path "/678ed6a7-73b5-414a-90da-5837647f5dd4/ba6f5248-4cb0-41f9-9534-0fba5bdbe75a/5ea1834a-1a07-4ed6-b43f-29b915030248"
+          (reference "R5") (unit 1)
+        )
+        (path "/678ed6a7-73b5-414a-90da-5837647f5dd4/ba6f5248-4cb0-41f9-9534-0fba5bdbe75a/84feea92-9e39-46cb-b5a7-5207e1eba94b"
+          (reference "R6") (unit 1)
+        )
+        (path "/678ed6a7-73b5-414a-90da-5837647f5dd4/ba6f5248-4cb0-41f9-9534-0fba5bdbe75a/4ec654a5-e9aa-4cd0-b4c8-093fac62fd4b"
+          (reference "R15") (unit 1)
+        )
+        (path "/678ed6a7-73b5-414a-90da-5837647f5dd4/ba6f5248-4cb0-41f9-9534-0fba5bdbe75a/3e7c86be-1ea7-4de9-ad71-2b4bfc847a48"
+          (reference "R16") (unit 1)
+        )
+        (path "/678ed6a7-73b5-414a-90da-5837647f5dd4/a3a78077-6b53-4c9d-ba53-5da8cf684a1d"
+          (reference "R68") (unit 1)
+        )
+      )
+    )
+  )
   (symbol (lib_id "Device:C_Small") (at 166.37 35.56 180) (unit 1)
     (in_bom yes) (on_board yes) (dnp no)
@@
         )
       )
+    )
+  )
+  (symbol (lib_id "Device:LED_Small") (at 45.72 104.14 0) (unit 1)
+    (in_bom yes) (on_board yes) (dnp no) (fields_autoplaced)
+    (property "Reference" "D2" (at 45.7835 99.06 0)
+      (effects (font (size 1.27 1.27)))
+    )
+    (property "Value" "LED_Small" (at 45.7835 101.6 0)
+      (effects (font (size 1.27 1.27)))
+    )
+    (property "Footprint" "LED_SMD:LED_0603_1608Metric_Pad1.05x0.95mm_HandSolder" (at 45.72 104.14 90)
+      (effects (font (size 1.27 1.27)) hide)
+    )
+    (property "Datasheet" "~" (at 45.72 104.14 90)
+      (effects (font (size 1.27 1.27)) hide)
+    )
+    (property "Part Number" "150060VS75000 " (at 45.72 104.14 0)
+      (effects (font (size 1.27 1.27)) hide)
+    )
+    (pin "1")
+    (pin "2")
+    (instances
+      (project "Power Module Rev 5"
+        (path "/678ed6a7-73b5-414a-90da-5837647f5dd4/a3a78077-6b53-4c9d-ba53-5da8cf684a1d"
+          (reference "D2") (unit 1)
+        )
+      )

Commit message: Board Update and Gerbers
Parts:
- removed Y1: Crystal_Small, Crystal:Crystal_SMD_5032-2Pin_5.0x3.2mm, symbol Device:Crystal_Small
- added Y3: 8MHz, Crystal:Crystal_SMD_5032-4Pin_5.0x3.2mm, symbol Device:Crystal_GND24_Small
- C13: value ~ -> 10pF
- Y2: value Crystal_Small -> 32.768kHz; footprint Crystal:Crystal_SMD_5032-2Pin_5.0x3.2mm -> Crystal:Crystal_SMD_3215-2Pin_3.2x1.5mm
Connections:
- net GND: now also Y3.2, Y3.4
- net at C13.2, U17.6 (PF1): now also Y3.3
- net at C13.2, U17.5 (PF0): now also Y3.1
