File: Board/Power Module Rev 5/Power Module Rev 5.kicad_pcb (KiCad board)
At the start: 4 copper layers, 76.2 x 101.6 mm, 133 parts, among them J1 9-6437287-8, J2 Conn_ARM_SWD_TagConnect_TC203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, J3 Conn_01x16_Pin, U1 STM32G491CCUx, U10 BTS7002-1EPP, U11 MCP2558FD-xMF, U12 BTS7008-2EPA, U13 BTS7008-2EPA, U14 TPS2116DRLR, U15 NCP167BMX330TBG, U16 PLMR38010FSQDDARQ1, U2 L9966CB-TR, U3 BTS7002-1EPP, U4 BTS7002-1EPP, U5 BTS7002-1EPP, U7 BTS7002-1EPP, U8 PCA9685BS, U9 BTS7002-1EPP

Commit message: Board Update
Parts:
- removed R61: 10K, Resistor_SMD:R_0603_1608Metric_Pad0.98x0.95mm_HandSolder
- removed U15: NCP167BMX330TBG, Package_DFN_QFN:OnSemi_XDFN4-1EP_1.0x1.0mm_EP0.52x0.52mm
- added C49: ~, Capacitor_SMD:C_0603_1608Metric_Pad1.08x0.95mm_HandSolder, F.Cu at (65.4, 48.1)
- added C50: ~, Capacitor_SMD:C_0603_1608Metric_Pad1.08x0.95mm_HandSolder, F.Cu at (65.4, 50.6)
- added FB1: FerriteBead_Small, Resistor_SMD:R_0603_1608Metric_Pad0.98x0.95mm_HandSolder, F.Cu at (71.1, 38.7)
- added J4: USB_C_Receptacle_USB2.0, Connector_USB:USB_C_Receptacle_JAE_DX07S016JA1R1500, F.Cu at (100.5, 33.3)
- added R66: 5.1K, Resistor_SMD:R_0603_1608Metric_Pad0.98x0.95mm_HandSolder, F.Cu at (108.1, 33.2)
- added R67: 5.1K, Resistor_SMD:R_0603_1608Metric_Pad0.98x0.95mm_HandSolder, F.Cu at (108.1, 35.7)
- added U17: STM32G491CEUx, Package_DFN_QFN:QFN-48-1EP_7x7mm_P0.5mm_EP5.6x5.6mm, F.Cu at (121.0, 65.5)
- added Y1: Crystal_Small, Crystal:Crystal_SMD_5032-2Pin_5.0x3.2mm, F.Cu at (59.8, 41.5)
- added Y2: Crystal_Small, Crystal:Crystal_SMD_5032-2Pin_5.0x3.2mm, F.Cu at (59.8, 46.4)
- C18, C19: value 6.8nF -> ~
- U1: value STM32G491CCUx -> AP2112K-3.3; footprint Package_DFN_QFN:QFN-48-1EP_7x7mm_P0.5mm_EP5.6x5.6mm -> Package_TO_SOT_SMD:SOT-23-5
- moved C18 133.8 mm to (65.4, 43.1)
- moved C19 133.3 mm to (65.4, 45.6)
- moved R57 122.9 mm to (146.8, 87.5), turned to -90 degrees
- moved R56 120.5 mm to (144.5, 84.7), turned to -90 degrees
- moved R55 119.6 mm to (143.0, 84.7), turned to -90 degrees
- moved U8 117.9 mm to (142.3, 90.2)
- moved C21 116.3 mm to (141.1, 84.7), turned to -90 degrees
- moved R43 77.2 mm to (125.2, 73.8), turned to 90 degrees
- moved R19 74.9 mm to (122.2, 73.8)
- moved C33 74.8 mm to (126.7, 73.8), turned to -90 degrees
- moved C29 72.1 mm to (123.7, 73.8), turned to -90 degrees
- moved C12 69.3 mm to (92.6, 119.3), turned to 180 degrees
- moved C6 69.0 mm to (92.6, 110.6), turned to 180 degrees
- moved C13 68.9 mm to (161.4, 118.2), turned to 0 degrees
- moved C15 68.9 mm to (161.4, 113.8), turned to 0 degrees
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Connections:
- C11 pad 1: Output7 -> Input3
- C12 pad 1: Output3 -> Input2
- C13 pad 1: Output2 -> Input1
- C14 pad 1: Output10 -> Output6
- C15 pad 1: L6699-IO3 -> Output4
- C16 pad 1: L6699-IO2 -> Output10
- C17 pad 1: L6699-IO1 -> Output9
- C18 pad 1: L6699-IO15 -> GND
- C18 pad 2: GND -> Net-(U17-PF1)
- C19 pad 1: L6699-IO14 -> GND
- C19 pad 2: GND -> Net-(U17-PF0)
- C20 pad 1: Output1 -> Output3
- C6 pad 1: Output9 -> Output5
- C7 pad 1: Output6 -> Output1
- C8 pad 1: Output5 -> Output2
- C9 pad 1: Output4 -> Output7
- D1 pad 1: Can- -> Can+
- D1 pad 2: Can+ -> Can-
- J1 pad 22: L6699-IO1 -> Input1
- J1 pad 23: L6699-IO2 -> Input2
- J1 pad 24: L6699-IO3 -> Input3
- J2 pad 1: unconnected-(J2-VCC-Pad1) -> +3.3V
- J2 pad 2: unconnected-(J2-SWDIO-Pad2) -> /Mcu/SWDIO
- J2 pad 3: unconnected-(J2-~{RESET}-Pad3) -> /Mcu/RESET
- J2 pad 4: unconnected-(J2-SWCLK-Pad4) -> /Mcu/SWCLK
- J2 pad 5: unconnected-(J2-GND-Pad5) -> GND
- J2 pad 6: unconnected-(J2-SWO-Pad6) -> /Mcu/SWO
- R23 pad 2: /High Side Drivers/Den2 -> Den2
- R27 pad 2: /High Side Drivers/Den5 -> Den5
- R4 pad 2: L6699-Sclk -> SPI1_Sclk
- R42 pad 2: Den9-10 -> /High Side Drivers/Den9-10
- R53 pad 2: Dsel9-10 -> /High Side Drivers/Dsel9-10
- R7 pad 2: L6699-Cs -> SPI1_SS1
- R8 pad 2: L6699-Mosi -> SPI1_Mosi
- R9 pad 2: L6699-Miso -> SPI1_Miso
- U1 pad 1: unconnected-(U1-VBAT-Pad1) -> +5V
- U1 pad 2: unconnected-(U1-PC13-Pad2) -> GND
- U1 pad 3: unconnected-(U1-PC14-Pad3) -> +5V
- U1 pad 5: unconnected-(U1-PF0-Pad5) -> +3.3V
- U2 pad 17: Output1 -> Output3
- U2 pad 18: L6699-IO14 -> unconnected-(U2-IO_14-Pad18)
- U2 pad 19: L6699-IO15 -> unconnected-(U2-IO_15-Pad19)
- U2 pad 20: L6699-IO1 -> Output9
- U2 pad 21: L6699-IO2 -> Output10
- U2 pad 22: L6699-IO3 -> Output4
- U2 pad 23: Output10 -> Output6
- U2 pad 39: Output9 -> Output5
- U2 pad 40: Output6 -> Output1
- U2 pad 41: Output5 -> Output2
- U2 pad 42: Output4 -> Output7
- U2 pad 44: Output7 -> Input3
- U2 pad 45: Output3 -> Input2
- U2 pad 46: Output2 -> Input1
- U8 pad 10: /High Side Drivers/In8 -> /High Side Drivers/In6
- U8 pad 12: /High Side Drivers/In9 -> /High Side Drivers/Den3
- U8 pad 13: /High Side Drivers/In10 -> /High Side Drivers/In3
- U8 pad 14: /High Side Drivers/Den6 -> /High Side Drivers/Den4
- U8 pad 15: /High Side Drivers/Den5 -> /High Side Drivers/In4
- U8 pad 16: /High Side Drivers/Den4 -> /High Side Drivers/In10
- U8 pad 17: /High Side Drivers/Den3 -> /High Side Drivers/Dsel9-10
- U8 pad 18: /High Side Drivers/Den2 -> /High Side Drivers/Den9-10
- U8 pad 19: /High Side Drivers/Den1 -> /High Side Drivers/In9
- U8 pad 3: /High Side Drivers/In1 -> /High Side Drivers/In8
- U8 pad 4: /High Side Drivers/In2 -> /High Side Drivers/In7
- U8 pad 5: /High Side Drivers/In3 -> /High Side Drivers/In2
- U8 pad 6: /High Side Drivers/In4 -> /High Side Drivers/In5
- U8 pad 7: /High Side Drivers/In5 -> /High Side Drivers/Den1
- U8 pad 8: /High Side Drivers/In6 -> /High Side Drivers/In1
- U8 pad 9: /High Side Drivers/In7 -> /High Side Drivers/Den6
Routing:
- net Input1: track 0.00 -> 127.0 mm, vias 0 -> 1
- net GND: track 0.00 -> 99.2 mm, vias 0 -> 77
- net Output3: track 34.6 -> 113.1 mm, vias 1 -> 3
- net Output6: track 41.4 -> 119.1 mm
- net Output4: track 37.5 -> 114.2 mm
- net Output9: track 40.2 -> 115.7 mm
- net Output10: track 35.9 -> 111.3 mm
- net Input2: track 0.00 -> 73.5 mm, vias 0 -> 1
- net Input3: track 0.00 -> 69.5 mm, vias 0 -> 1
- net /High Side Drivers/In8: track 15.2 -> 79.9 mm
- net /High Side Drivers/In7: track 9.39 -> 72.7 mm
- net +5V: track 0.00 -> 62.7 mm, vias 0 -> 9
- net /High Side Drivers/In2: track 3.42 -> 65.8 mm
- net Net-(U13-IS): track 3.07 -> 65.4 mm, vias 0 -> 3
- net Can-: track 0.00 -> 56.1 mm, vias 0 -> 1
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- added copper zone on In1.Cu, net +12V
- added copper zone on F.Cu, net +3.3V
- added copper zone on In1.Cu, net +3.3V
- added copper zone on F.Cu, net +5V
- added copper zone on In1.Cu, net +5V
- added copper zone on F.Cu, net Ignition
- added copper zone on B.Cu, net Output1
- added copper zone on In1.Cu, net Output1
- added copper zone on In2.Cu, net Output1
- added copper zone on B.Cu, net Output10
- added copper zone on F.Cu, net Output10
- added copper zone on In2.Cu, net Output10
- added copper zone on B.Cu, net Output2
- added copper zone on F.Cu, net Output2
- added copper zone on In2.Cu, net Output2
- added copper zone on In1.Cu, net Output3
- added copper zone on In2.Cu, net Output3
- added copper zone on In2.Cu, net Output4
- added copper zone on B.Cu, net Output5
- added copper zone on F.Cu, net Output5
- added copper zone on In1.Cu, net Output5
- added copper zone on In2.Cu, net Output5
- added copper zone on In1.Cu, net Output6
- added copper zone on In2.Cu, net Output6
- added copper zone on B.Cu, net Output7
- added copper zone on F.Cu, net Output7
- added copper zone on In2.Cu, net Output7
- added copper zone on B.Cu, net Output8
- added copper zone on F.Cu, net Output8
- added copper zone on In2.Cu, net Output8
- added copper zone on B.Cu, net Output9
- added copper zone on F.Cu, net Output9
- added copper zone on In2.Cu, net Output9

Commit message: Board Update
Parts:
- added C51: 0.1uF, Capacitor_SMD:C_0603_1608Metric_Pad1.08x0.95mm_HandSolder, F.Cu at (131.4, 59.4)
- added C52: 0.1uF, Capacitor_SMD:C_0603_1608Metric_Pad1.08x0.95mm_HandSolder, F.Cu at (114.1, 59.5)
- added C53: 0.1uF, Capacitor_SMD:C_0603_1608Metric_Pad1.08x0.95mm_HandSolder, F.Cu at (123.7, 68.4)
- added C54: 0.1uF, Capacitor_SMD:C_0603_1608Metric_Pad1.08x0.95mm_HandSolder, F.Cu at (123.7, 69.9)
- added C55: 0.1uF, Capacitor_SMD:C_0603_1608Metric_Pad1.08x0.95mm_HandSolder, F.Cu at (111.9, 68.5)
- added C56: 1uF, Capacitor_SMD:C_0603_1608Metric_Pad1.08x0.95mm_HandSolder, F.Cu at (117.4, 56.0)
- added C57: 10nF, Capacitor_SMD:C_0603_1608Metric_Pad1.08x0.95mm_HandSolder, F.Cu at (117.4, 57.5)
- added R61: 10K, Resistor_SMD:R_0603_1608Metric_Pad0.98x0.95mm_HandSolder, F.Cu at (140.2, 59.4)
- added S1: B3U-1000P, digikey-footprints:Switch_Tactile_SMD_B3U-1000P, F.Cu at (147.8, 56.6)
- added S2: B3U-1000P, digikey-footprints:Switch_Tactile_SMD_B3U-1000P, F.Cu at (140.9, 56.6)
- added U6: MB85RS64, Package_SO:SSOP-8_3.9x5.05mm_P1.27mm, F.Cu at (133.5, 55.8)
- U17: footprint Package_DFN_QFN:QFN-48-1EP_7x7mm_P0.5mm_EP5.6x5.6mm -> Package_DFN_QFN:QFN-48-1EP_7x7mm_P0.5mm_EP5.6x5.6mm_ThermalVias
- U8: footprint Package_DFN_QFN:QFN-28-1EP_6x6mm_P0.65mm_EP4.25x4.25mm -> Package_DFN_QFN:QFN-28-1EP_6x6mm_P0.65mm_EP4.25x4.25mm_ThermalVias
- moved Y2 71.4 mm to (127.9, 67.8), turned to -90 degrees
- moved Y1 71.0 mm to (127.9, 61.5), turned to -90 degrees
- moved C49 69.0 mm to (131.4, 68.3), turned to 180 degrees
- moved C18 68.4 mm to (131.4, 60.9), turned to 180 degrees
- moved C19 68.1 mm to (131.4, 62.4), turned to 180 degrees
- moved C50 68.0 mm to (131.4, 66.9), turned to 180 degrees
- moved FB1 50.6 mm to (117.4, 58.9), turned to 180 degrees
- moved J2 39.0 mm to (102.4, 67.2), turned to 90 degrees
- moved R48 22.9 mm to (96.2, 62.6)
- moved C35 22.9 mm to (96.2, 64.1)
- moved R66 20.8 mm to (104.0, 53.6), turned to 180 degrees
- moved C27 20.8 mm to (96.2, 65.6)
- moved R17 19.8 mm to (96.2, 67.1)
- moved C30 19.4 mm to (96.2, 71.5), turned to 180 degrees
- moved R20 19.4 mm to (96.2, 72.9), turned to 0 degrees
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Connections:
- U17 pad 11: Is4 -> Is6
- U17 pad 12: SPI1_SS1 -> /Mcu/Memory_Hold
- U17 pad 16: unconnected-(U17-PC4-Pad16) -> /Mcu/SPI1_SS2
- U17 pad 17: /Mcu/SPI1_SS2 -> /Mcu/Memory_Wp
- U17 pad 18: Is5 -> Is7-8
- U17 pad 19: unconnected-(U17-PB2-Pad19) -> Power Switch Status
- U17 pad 2: L6699-Sync -> CanSilent
- U17 pad 22: Den5 -> unconnected-(U17-PB10-Pad22)
- U17 pad 24: Is6 -> Is2
- U17 pad 25: Is7-8 -> Is5
- U17 pad 26: Dsel7-8 -> unconnected-(U17-PB13-Pad26)
- U17 pad 27: Is9-10 -> Is1
- U17 pad 28: Den7-8 -> Den2
- U17 pad 29: unconnected-(U17-PC6-Pad29) -> Dsel7-8
- U17 pad 32: Pwm_Ctr_Enable -> Den7-8
- U17 pad 38: Power Switch Status -> Den5
- U17 pad 39: CanSilent -> SPI1_SS1
- U17 pad 45: unconnected-(U17-PB7-Pad45) -> L6699-Sync
- U17 pad 47: Den2 -> Pwm_Ctr_Enable
- U17 pad 8: Is1 -> Is9-10
- U17 pad 9: Is2 -> Is4
Routing:
- net SPI1_Miso: track 6.49 -> 79.3 mm, vias 0 -> 2
- net SPI1_Sclk: track 11.3 -> 79.8 mm, vias 0 -> 2
- net SPI1_Mosi: track 8.11 -> 76.1 mm, vias 0 -> 2
- net /Mcu/RESET: track 0.00 -> 59.2 mm, vias 0 -> 3
- net Pwm_Ctr_Enable: track 1.91 -> 48.9 mm, vias 0 -> 2
- net Den2: track 25.9 -> 68.3 mm, vias 2 -> 4
- net Den5: track 17.7 -> 59.6 mm, vias 2 -> 4
- net Dsel7-8: track 33.6 -> 75.3 mm, vias 2 -> 4
- net Den7-8: track 29.9 -> 71.5 mm, vias 2 -> 4
- net Power Switch Status: track 1.62 -> 40.0 mm
- net /Mcu/BOOT_0: track 0.00 -> 36.8 mm, vias 0 -> 2
- net Net-(U12-IS): track 33.1 -> 63.7 mm
- net GND: track 99.2 -> 129.7 mm, vias 77 -> 88
- net L6699-Sync: track 4.82 -> 31.9 mm, vias 0 -> 2
- net SDA: track 22.1 -> 49.1 mm, vias 2 -> 4
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
Commit message: Update Board
Parts:
- added C40: 100nF, Capacitor_SMD:C_0603_1608Metric_Pad1.08x0.95mm_HandSolder, F.Cu at (120.9, 87.9)
- added FB2: FerriteBead_Small, Resistor_SMD:R_0603_1608Metric_Pad0.98x0.95mm_HandSolder, F.Cu at (100.7, 57.6)
- moved R66 5.23 mm to (104.1, 58.8)
- moved R67 5.23 mm to (109.6, 58.8)
- moved J4 4.02 mm to (106.7, 52.3)
- moved Y1 0.08 mm to (127.8, 61.5)
Connections:
- J4 pad S1: unconnected-(J4-SHIELD-PadS1) -> /Mcu/Usb_Shield
Routing:
- net Usb 5V: track 0.00 -> 55.6 mm
- net GND: track 129.7 -> 139.1 mm, vias 88 -> 99
- net /Mcu/Usb D-: track 12.5 -> 18.6 mm
- net +12V: track 53.2 -> 47.6 mm, vias 3 -> 25
- net Net-(J4-CC1): track 0.00 -> 3.66 mm
- net Net-(J4-CC2): track 0.00 -> 3.62 mm
- net /Mcu/Usb D+: track 13.3 -> 16.9 mm
- net Output9: track 115.7 -> 114.3 mm, vias 1 -> 3
- net Output8: track 66.8 -> 65.5 mm, vias 1 -> 3
- net /Mcu/RESET: track 59.2 -> 58.6 mm
- net Output7: vias 1 -> 3
- net Output6: vias 1 -> 5
- net Output5: vias 1 -> 5
- net Output4: vias 1 -> 5
- net Output3: vias 3 -> 7
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- added copper zone on F.Cu, net /Mcu/Usb_Shield
- added copper zone on In1.Cu, net Output10
- added copper zone on In1.Cu, net Output2
- added copper zone on In1.Cu, net Output4
- added copper zone on In1.Cu, net Output7
- added copper zone on In1.Cu, net Output8
- added copper zone on In1.Cu, net Output9
Other:
- board size 76.2 x 101.6 mm -> 76.2 x 82.6 mm
