File: Board/Power Module Rev 5/Power Module Rev 5.kicad_pcb (KiCad board)
At the start: 4 copper layers, 76.2 x 82.6 mm, 153 parts, among them J1 9-6437287-8, J2 Conn_ARM_SWD_TagConnect_TC203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, J3 Conn_01x16_Pin, J4 USB_C_Receptacle_USB2.0, U1 AP2112K-3.3, U10 BTS7002-1EPP, U11 MCP2558FD-xMF, U12 BTS7008-2EPA, U13 BTS7008-2EPA, U14 TPS2116DRLR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

Commit message: Update config and renames on schematic
Connections:
- net /Mcu/SPI1_SS2 renamed /Mcu/SPI1_SS_Memory
- net Power Switch Status renamed PowerSwitchStatus
- net SPI1_SS1 renamed SPI1_SS_L9966
Routing:
- net GND: vias 99 -> 107
- net +12V: vias 25 -> 28
- added copper zone on B.Cu, net GND
Other:
- board text added: "BOOT_0"
- board text added: "Power Module - Rev 5 2023"
- board text added: "RESET"
