File: Board/Power Module Rev 5/HighSideDrivers.kicad_sch (KiCad schematic)
At the start: 5 parts, among them U14 PCA9685BS

Commit message: Update Board
Connections:
- net Den1: now also U14.7 (LED4); no longer U14.19 (LED15)
- net Den2: no longer U14.18 (LED14)
- net Den3: now also U14.12 (LED8); no longer U14.17 (LED13)
- net Den4: now also U14.14 (LED10); no longer U14.16 (LED12)
- net Den5: no longer U14.15 (LED11)
- net Den6: now also U14.9 (LED6); no longer U14.14 (LED10)
- net Den9-10: now also U14.18 (LED14)
- net Dsel9-10: now also U14.17 (LED13)
- net In1: now also U14.8 (LED5); no longer U14.3 (LED0)
- net In10: now also U14.16 (LED12); no longer U14.13 (LED9)
- net In2: now also U14.5 (LED2); no longer U14.4 (LED1)
- net In3: now also U14.13 (LED9); no longer U14.5 (LED2)
- net In4: now also U14.15 (LED11); no longer U14.6 (LED3)
- net In5: now also U14.6 (LED3); no longer U14.7 (LED4)
- net In6: now also U14.10 (LED7); no longer U14.8 (LED5)
- net In7: now also U14.4 (LED1); no longer U14.9 (LED6)
- net In8: now also U14.3 (LED0); no longer U14.10 (LED7)
- net In9: now also U14.19 (LED15); no longer U14.12 (LED8)
Changed lines of the file:
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@@
     (stroke (width 0) (type default))
   )
-  (label "In4" (at 87.63 49.53 0) (fields_autoplaced)
+  (label "Den9-10" (at 87.63 77.47 0) (fields_autoplaced)
+    (effects (font (size 1.27 1.27)) (justify left bottom))
+  )
+  (label "In4" (at 87.63 69.85 0) (fields_autoplaced)
+    (effects (font (size 1.27 1.27)) (justify left bottom))
+  )
+  (label "In8" (at 87.63 41.91 0) (fields_autoplaced)
     (effects (font (size 1.27 1.27)) (justify left bottom))
   )
@@
     (effects (font (size 1.27 1.27)) (justify right bottom))
   )
-  (label "In8" (at 87.63 59.69 0) (fields_autoplaced)
-    (effects (font (size 1.27 1.27)) (justify left bottom))
-  )
   (label "In6" (at 219.71 81.28 180) (fields_autoplaced)
     (effects (font (size 1.27 1.27)) (justify right bottom))
   )
-  (label "Den4" (at 87.63 72.39 0) (fields_autoplaced)
-    (effects (font (size 1.27 1.27)) (justify left bottom))
-  )
-  (label "In9" (at 87.63 62.23 0) (fields_autoplaced)
-    (effects (font (size 1.27 1.27)) (justify left bottom))
-  )
-  (label "In1" (at 87.63 41.91 0) (fields_autoplaced)
+  (label "In7" (at 87.63 44.45 0) (fields_autoplaced)
+    (effects (font (size 1.27 1.27)) (justify left bottom))
+  )
+  (label "Den4" (at 87.63 67.31 0) (fields_autoplaced)
+    (effects (font (size 1.27 1.27)) (justify left bottom))
+  )
+  (label "In9" (at 87.63 80.01 0) (fields_autoplaced)
+    (effects (font (size 1.27 1.27)) (justify left bottom))
+  )
+  (label "In1" (at 87.63 54.61 0) (fields_autoplaced)
     (effects (font (size 1.27 1.27)) (justify left bottom))
   )
@@
     (effects (font (size 1.27 1.27)) (justify right bottom))
   )
-  (label "Den2" (at 87.63 77.47 0) (fields_autoplaced)
-    (effects (font (size 1.27 1.27)) (justify left bottom))
-  )
-  (label "In6" (at 87.63 54.61 0) (fields_autoplaced)
-    (effects (font (size 1.27 1.27)) (justify left bottom))
+  (label "In7" (at 143.51 132.08 180) (fields_autoplaced)
+    (effects (font (size 1.27 1.27)) (justify right bottom))
+  )
+  (label "In6" (at 87.63 59.69 0) (fields_autoplaced)
+    (effects (font (size 1.27 1.27)) (justify left bottom))
+  )
+  (label "Den9-10" (at 217.17 137.16 180) (fields_autoplaced)
+    (effects (font (size 1.27 1.27)) (justify right bottom))
   )
   (label "In9" (at 217.17 132.08 180) (fields_autoplaced)
@@
     (effects (font (size 1.27 1.27)) (justify right bottom))
   )
-  (label "Den1" (at 87.63 80.01 0) (fields_autoplaced)
-    (effects (font (size 1.27 1.27)) (justify left bottom))
-  )
-  (label "In5" (at 87.63 52.07 0) (fields_autoplaced)
-    (effects (font (size 1.27 1.27)) (justify left bottom))
-  )
-  (label "Den6" (at 87.63 67.31 0) (fields_autoplaced)
+  (label "Den1" (at 87.63 52.07 0) (fields_autoplaced)
+    (effects (font (size 1.27 1.27)) (justify left bottom))
+  )
+  (label "In5" (at 87.63 49.53 0) (fields_autoplaced)
+    (effects (font (size 1.27 1.27)) (justify left bottom))
+  )
+  (label "Den6" (at 87.63 57.15 0) (fields_autoplaced)
     (effects (font (size 1.27 1.27)) (justify left bottom))
   )
@@
     (effects (font (size 1.27 1.27)) (justify right bottom))
   )
-  (label "In10" (at 87.63 64.77 0) (fields_autoplaced)
-    (effects (font (size 1.27 1.27)) (justify left bottom))
-  )
-  (label "Den5" (at 87.63 69.85 0) (fields_autoplaced)
-    (effects (font (size 1.27 1.27)) (justify left bottom))
+  (label "In8" (at 143.51 134.62 180) (fields_autoplaced)
+    (effects (font (size 1.27 1.27)) (justify right bottom))
+  )
+  (label "In10" (at 87.63 72.39 0) (fields_autoplaced)
+    (effects (font (size 1.27 1.27)) (justify left bottom))
+  )
+  (label "Dsel9-10" (at 217.17 139.7 180) (fields_autoplaced)
+    (effects (font (size 1.27 1.27)) (justify right bottom))
   )
   (label "In5" (at 219.71 53.34 180) (fields_autoplaced)
     (effects (font (size 1.27 1.27)) (justify right bottom))
   )
-  (label "In2" (at 87.63 44.45 0) (fields_autoplaced)
+  (label "In2" (at 87.63 46.99 0) (fields_autoplaced)
     (effects (font (size 1.27 1.27)) (justify left bottom))
   )
@@
     (effects (font (size 1.27 1.27)) (justify right bottom))
   )
-  (label "Den3" (at 87.63 74.93 0) (fields_autoplaced)
-    (effects (font (size 1.27 1.27)) (justify left bottom))
-  )
-  (label "Den5" (at 219.71 55.88 180) (fields_autoplaced)
-    (effects (font (size 1.27 1.27)) (justify right bottom))
+  (label "Den3" (at 87.63 62.23 0) (fields_autoplaced)
+    (effects (font (size 1.27 1.27)) (justify left bottom))
   )
   (label "In3" (at 143.51 80.01 180) (fields_autoplaced)
     (effects (font (size 1.27 1.27)) (justify right bottom))
   )
-  (label "In7" (at 143.51 132.08 180) (fields_autoplaced)
-    (effects (font (size 1.27 1.27)) (justify right bottom))
-  )
-  (label "In7" (at 87.63 57.15 0) (fields_autoplaced)
-    (effects (font (size 1.27 1.27)) (justify left bottom))
-  )
-  (label "In3" (at 87.63 46.99 0) (fields_autoplaced)
-    (effects (font (size 1.27 1.27)) (justify left bottom))
-  )
-  (label "In8" (at 143.51 134.62 180) (fields_autoplaced)
-    (effects (font (size 1.27 1.27)) (justify right bottom))
-  )
-  (label "Den2" (at 143.51 57.15 180) (fields_autoplaced)
-    (effects (font (size 1.27 1.27)) (justify right bottom))
+  (label "In3" (at 87.63 64.77 0) (fields_autoplaced)
+    (effects (font (size 1.27 1.27)) (justify left bottom))
+  )
+  (label "Dsel9-10" (at 87.63 74.93 0) (fields_autoplaced)
+    (effects (font (size 1.27 1.27)) (justify left bottom))
   )
   (label "In2" (at 143.51 54.61 180) (fields_autoplaced)
@@
     (effects (font (size 1.27 1.27)) (justify right))
     (property "Intersheetrefs" "${INTERSHEET_REFS}" (at 133.1052 137.16 0)
+      (effects (font (size 1.27 1.27)) (justify right) hide)
+    )
+  )
+  (global_label "Den5" (shape input) (at 219.71 55.88 180) (fields_autoplaced)
+    (effects (font (size 1.27 1.27)) (justify right))
+    (property "Intersheetrefs" "${INTERSHEET_REFS}" (at 212.0871 55.88 0)
       (effects (font (size 1.27 1.27)) (justify right) hide)
     )
@@
     )
   )
-  (global_label "Dsel9-10" (shape input) (at 217.17 139.7 180) (fields_autoplaced)
-    (effects (font (size 1.27 1.27)) (justify right))
-    (property "Intersheetrefs" "${INTERSHEET_REFS}" (at 205.0114 139.7 0)
-      (effects (font (size 1.27 1.27)) (justify right) hide)
-    )
-  )
   (global_label "Output4" (shape input) (at 257.81 29.21 0) (fields_autoplaced)
     (effects (font (size 1.27 1.27)) (justify left))
@@
     )
   )
-  (global_label "Den9-10" (shape input) (at 217.17 137.16 180) (fields_autoplaced)
-    (effects (font (size 1.27 1.27)) (justify right))
-    (property "Intersheetrefs" "${INTERSHEET_REFS}" (at 205.5557 137.16 0)
-      (effects (font (size 1.27 1.27)) (justify right) hide)
-    )
+  (global_label "Den2" (shape input) (at 143.51 57.15 180) (fields_autoplaced)
+    (effects (font (size 1.27 1.27)) (justify right))
+    (property "Intersheetrefs" "${INTERSHEET_REFS}" (at 135.8871 57.15 0)
+      (effects (font (size 1.27 1.27)) (justify right) hide)
+    )

Commit message: Board Update
Parts:
- U14: footprint Package_DFN_QFN:QFN-28-1EP_6x6mm_P0.65mm_EP4.25x4.25mm -> Package_DFN_QFN:QFN-28-1EP_6x6mm_P0.65mm_EP4.25x4.25mm_ThermalVias
Changed lines of the file:
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@@
       (effects (font (size 1.27 1.27)) (justify left))
     )
-    (property "Footprint" "Package_DFN_QFN:QFN-28-1EP_6x6mm_P0.65mm_EP4.25x4.25mm" (at 66.675 84.455 0)
+    (property "Footprint" "Package_DFN_QFN:QFN-28-1EP_6x6mm_P0.65mm_EP4.25x4.25mm_ThermalVias" (at 66.675 84.455 0)
       (effects (font (size 1.27 1.27)) (justify left) hide)
     )

Commit message: Board Update and Gerbers
Parts:
- R2, R3: value 4K7 -> 4.7K
Changed lines of the file:
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@@
       (effects (font (size 1.27 1.27)) (justify left))
     )
-    (property "Value" "4K7" (at 31.9786 37.973 0)
+    (property "Value" "4.7K" (at 31.9786 37.973 0)
       (effects (font (size 1.27 1.27)) (justify left))
     )
@@
       (effects (font (size 1.27 1.27)) (justify left))
     )
-    (property "Value" "4K7" (at 38.3286 37.973 0)
+    (property "Value" "4.7K" (at 38.3286 37.973 0)
       (effects (font (size 1.27 1.27)) (justify left))
     )
