File: Board/Power Module Rev 5/SingleOutput.kicad_sch (KiCad schematic)
At the start: 8 parts, among them U3 BTS7002-1EPP

Commit message: Board Update and Gerbers
Parts:
- C34: value 100nF -> 0.1uF
Changed lines of the file:
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@@
       (effects (font (size 1.27 1.27)) (justify left))
     )
-    (property "Value" "100nF" (at 124.46 45.0913 0)
+    (property "Value" "0.1uF" (at 124.46 45.0913 0)
       (effects (font (size 1.27 1.27)) (justify left))
     )
