File: Board/Adc Adapter/Adc Adapter.kicad_pcb (KiCad board)
At the start: 2 copper layers, 29.9 x 15.9 mm, 22 parts, among them J1 Conn_01x01_Pin, U1 LM324DT

Commit message: Adc adapter gerber outputs
Other:
- board size 29.9 x 15.9 mm -> 24.3 x 14.5 mm
Changed lines of the file:
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@@
       (plot_on_all_layers_selection 0x0000000_00000000)
       (disableapertmacros false)
-      (usegerberextensions false)
-      (usegerberattributes true)
-      (usegerberadvancedattributes true)
-      (creategerberjobfile true)
+      (usegerberextensions true)
+      (usegerberattributes false)
+      (usegerberadvancedattributes false)
+      (creategerberjobfile false)
       (dashed_line_dash_ratio 12.000000)
       (dashed_line_gap_ratio 3.000000)
@@
       (psa4output false)
       (plotreference true)
-      (plotvalue true)
+      (plotvalue false)
       (plotinvisibletext false)
       (sketchpadsonfab false)
-      (subtractmaskfromsilk false)
+      (subtractmaskfromsilk true)
       (outputformat 1)
       (mirror false)
-      (drillshape 1)
+      (drillshape 0)
       (scaleselection 1)
-      (outputdirectory "")
+      (outputdirectory "plots/")
     )
   )
@@
     (property "ki_keywords" "R resistor")
     (attr smd)
-    (fp_text reference "R4" (at 0 -1.43) (layer "F.SilkS")
+    (fp_text reference "R4" (at 2.667 0.154213) (layer "F.SilkS")
         (effects (font (size 1 1) (thickness 0.15)))
     )
@@
     (property "ki_keywords" "R resistor")
     (attr smd)
-    (fp_text reference "R3" (at 0 -1.43) (layer "F.SilkS")
+    (fp_text reference "R3" (at 2.6416 0.078013) (layer "F.SilkS")
         (effects (font (size 1 1) (thickness 0.15)))
     )
@@
     (property "ki_keywords" "R resistor")
     (attr smd)
-    (fp_text reference "R12" (at 0 -1.43) (layer "F.SilkS")
+    (fp_text reference "R12" (at -3.1261 0.166916) (layer "F.SilkS")
         (effects (font (size 1 1) (thickness 0.15)))
     )
@@
     (property "ki_keywords" "capacitor cap")
     (attr smd)
-    (fp_text reference "C4" (at 0 -1.43) (layer "F.SilkS")
+    (fp_text reference "C4" (at 2.6162 0.128813) (layer "F.SilkS")
         (effects (font (size 1 1) (thickness 0.15)))
     )
@@
     (property "ki_keywords" "capacitor cap")
     (attr smd)
-    (fp_text reference "C6" (at 0 -1.43) (layer "F.SilkS")
+    (fp_text reference "C6" (at 2.794 0.0508) (layer "F.SilkS")
         (effects (font (size 1 1) (thickness 0.15)))
     )
@@
     (property "ki_keywords" "R resistor")
     (attr smd)
-    (fp_text reference "R9" (at 0 -1.43) (layer "F.SilkS")
+    (fp_text reference "R9" (at -2.6689 0.097968) (layer "F.SilkS")
         (effects (font (size 1 1) (thickness 0.15)))
     )
@@
     (property "ki_keywords" "R resistor")
     (attr smd)
-    (fp_text reference "R1" (at 0 -1.43) (layer "F.SilkS")
+    (fp_text reference "R1" (at 2.6924 0.179613) (layer "F.SilkS")
         (effects (font (size 1 1) (thickness 0.15)))
     )
@@
     (property "ki_keywords" "R resistor")
     (attr smd)
-    (fp_text reference "R8" (at 0 -1.43) (layer "F.SilkS")
+    (fp_text reference "R8" (at 2.6689 -0.083458) (layer "F.SilkS")
         (effects (font (size 1 1) (thickness 0.15)))
     )
@@
     (property "ki_keywords" "capacitor cap")
     (attr smd)
-    (fp_text reference "C8" (at 0 -1.43) (layer "F.SilkS")
+    (fp_text reference "C8" (at -2.6162 0.127) (layer "F.SilkS")
         (effects (font (size 1 1) (thickness 0.15)))
     )
@@
     (property "ki_keywords" "capacitor cap")
     (attr smd)
-    (fp_text reference "C7" (at 0 -1.43) (layer "F.SilkS")
+    (fp_text reference "C7" (at -2.7432 0.1778) (layer "F.SilkS")
         (effects (font (size 1 1) (thickness 0.15)))
     )
@@
     (property "ki_keywords" "connector")
     (attr through_hole)
-    (fp_text reference "J1" (at 0 -2.06) (layer "F.SilkS")
+    (fp_text reference "J1" (at 0 -2.06) (layer "F.SilkS") hide
         (effects (font (size 1 1) (thickness 0.15)))
     )
@@
     (property "ki_keywords" "R resistor")
     (attr smd)
-    (fp_text reference "R10" (at 0 -1.43) (layer "F.SilkS")
+    (fp_text reference "R10" (at -3.0753 0.112484) (layer "F.SilkS")
         (effects (font (size 1 1) (thickness 0.15)))
     )
@@
     (property "ki_keywords" "497-1580-1-ND")
     (attr smd)
-    (fp_text reference "U1" (at 0 -4.79) (layer "F.SilkS")
+    (fp_text reference "U1" (at 0 -4.79) (layer "F.SilkS") hide
         (effects (font (size 1 1) (thickness 0.15)))
     )
@@
     (property "ki_keywords" "capacitor cap")
     (attr smd)
-    (fp_text reference "C3" (at 0 -1.43) (layer "F.SilkS")
+    (fp_text reference "C3" (at 2.6416 0.078013) (layer "F.SilkS")
         (effects (font (size 1 1) (thickness 0.15)))
     )
@@
     (property "ki_keywords" "R resistor")
     (attr smd)
-    (fp_text reference "R11" (at 0 -1.43) (layer "F.SilkS")
+    (fp_text reference "R11" (at -3.1515 0.0508) (layer "F.SilkS")
         (effects (font (size 1 1) (thickness 0.15)))
     )
@@
     (property "ki_keywords" "R resistor")
     (attr smd)
-    (fp_text reference "R5" (at 0 -1.43) (layer "F.SilkS")
+    (fp_text reference "R5" (at 2.6181 -0.09071) (layer "F.SilkS")
         (effects (font (size 1 1) (thickness 0.15)))
     )
@@
     (property "ki_keywords" "R resistor")
     (attr smd)
-    (fp_text reference "R7" (at 0 -1.43) (layer "F.SilkS")
+    (fp_text reference "R7" (at 2.6435 -0.145142) (layer "F.SilkS")
         (effects (font (size 1 1) (thickness 0.15)))
     )
@@
     (property "ki_keywords" "R resistor")
     (attr smd)
-    (fp_text reference "R6" (at 0 -1.43) (layer "F.SilkS")
+    (fp_text reference "R6" (at 2.6689 -0.079826) (layer "F.SilkS")
         (effects (font (size 1 1) (thickness 0.15)))
     )
@@
     (property "ki_keywords" "capacitor cap")
     (attr smd)
-    (fp_text reference "C1" (at 0 -1.43) (layer "F.SilkS")
+    (fp_text reference "C1" (at 2.6924 0.078013) (layer "F.SilkS")
         (effects (font (size 1 1) (thickness 0.15)))
     )
@@
     (property "ki_keywords" "capacitor cap")
     (attr smd)
-    (fp_text reference "C2" (at 0 -1.43) (layer "F.SilkS")
+    (fp_text reference "C2" (at 2.667 0.128813) (layer "F.SilkS")
         (effects (font (size 1 1) (thickness 0.15)))
     )
@@
     (property "ki_keywords" "capacitor cap")
     (attr smd)
-    (fp_text reference "C5" (at 0 -1.43) (layer "F.SilkS")
+    (fp_text reference "C5" (at 2.7686 0.1778) (layer "F.SilkS")
         (effects (font (size 1 1) (thickness 0.15)))
     )
@@
     (property "ki_keywords" "R resistor")
     (attr smd)
-    (fp_text reference "R2" (at 0 -1.43) (layer "F.SilkS")
+    (fp_text reference "R2" (at 2.6416 0.154213) (layer "F.SilkS")
         (effects (font (size 1 1) (thickness 0.15)))
     )
@@
       (net 3 "Is2") (pintype "passive"))
   )
-  (gr_rect (start 104.1146 59.9948) (end 134.0358 75.9206)
+  (gr_rect (start 104.8766 59.9948) (end 129.2098 74.5236)
     (stroke (width 0.1) (type default)) (fill none) (layer "Edge.Cuts"))
-  (dimension (type aligned) (layer "F.Cu")
-    (pts (xy 104.3178 74.3204) (xy 129.5146 74.168))
-    (height 5.516429)
-    (gr_text "0.9920 in" (at 116.938678 77.960561 0.3465428277) (layer "F.Cu")
-      (effects (font (size 1.5 1.5) (thickness 0.3)))
-    )
-    (format (prefix "") (suffix "") (units 3) (units_format 1) (precision 4))
-    (style (thickness 0.2) (arrow_length 1.27) (text_position_mode 0) (extension_height 0.58642) (extension_offset 0.5) keep_text_aligned)
-  )
-  (dimension (type aligned) (layer "F.Cu")
-    (pts (xy 108.5088 74.5236) (xy 114.1984 74.549))
-    (height 2.090548)
-    (gr_text "0.2240 in" (at 111.352303 74.826845 359.744217) (layer "F.Cu")
-      (effects (font (size 1.5 1.5) (thickness 0.3)))
-    )
-    (format (prefix "") (suffix "") (units 3) (units_format 1) (precision 4))
-    (style (thickness 0.2) (arrow_length 1.27) (text_position_mode 0) (extension_height 0.58642) (extension_offset 0.5) keep_text_aligned)
-  )
   (segment (start 128.3418 64.3592) (end 128.3418 68.4842) (width 0.1524) (layer "F.Cu") (net 1))
   (segment (start 105.9191 70.178387) (end 105.9191 70.244387) (width 0.1524) (layer "F.Cu") (net 1))
